File: Playgrounds/ESP32 Breakouts Playground/ESP32 Breakouts Playground.kicad_pcb (KiCad board)
At the start: 2 copper layers, 117 parts, among them J1 Conn_01x02_Socket, J10 Conn_01x03_Socket, J11 Conn_01x03_Socket, J12 Conn_01x11_Socket, J13 Conn_01x02_Socket, J14 Screw_Terminal_01x04, J15 Conn_01x06_Socket, J16 Conn_01x05_Socket, J17 USB4105-GF-A, J18 Conn_01x03_Socket, J19 Conn_01x02_Socket, J2 Conn_01x02_Socket, J20 Conn_01x02_Socket, J21 Conn_01x06_Socket, J22 Conn_01x05_Socket, J23 Conn_01x02_Socket, J24 Conn_01x06_Socket, J25 Conn_01x06_Socket, J26 Conn_01x04_Socket, J27 RJ45_Amphenol_RJMG1BD3B8K1ANR, J3 Conn_01x02_Socket, J4 Conn_01x02_Socket, J5 Conn_01x02_Socket, J6 Conn_01x06_Socket, J7 Conn_01x11_Socket, J8 Conn_01x02_Socket, J9 Conn_01x12_Socket, SW1 SW_RST, SW2 SW_BOOT, U1 AP63203WU, U2 FT230XS-R, U3 ESP32-S3-WROOM-1, U4 MAX31865xAP, U5 LAN8720A

Commit message: Finished routing
Routing:
- net GND: track 575.8 -> 657.4 mm
- net Net-(J27-LEDY_A): track 0.00 -> 64.9 mm, vias 0 -> 1
- net Net-(J26-Pin_1): track 0.00 -> 64.0 mm
- net Net-(J26-Pin_3): track 0.00 -> 51.9 mm
- net Net-(J25-Pin_3): track 0.00 -> 43.9 mm, vias 0 -> 2
- net Net-(J25-Pin_4): track 0.00 -> 42.3 mm, vias 0 -> 3
- net Net-(J25-Pin_6): track 0.00 -> 38.4 mm, vias 0 -> 1
- net Net-(J27-LEDG_A): track 0.00 -> 35.4 mm
- net Net-(J25-Pin_5): track 0.00 -> 33.8 mm, vias 0 -> 1
- net Net-(J25-Pin_2): track 0.00 -> 33.7 mm
- net Net-(J25-Pin_1): track 0.00 -> 24.0 mm
- net Net-(J26-Pin_2): track 0.00 -> 7.05 mm
- net Net-(J26-Pin_4): track 0.00 -> 4.12 mm
Other:
- board outline added: 203.1 x 108.1 mm

Commit message: ordered today jlcpcb
Routing:
- added copper zone on B.Cu, net GND
- added copper zone on F.Cu, net GND
